File: hardware/DISPLAY.kicad_sch (KiCad schematic)
At the start: 16 parts, among them U10 LTC-5723HR, U11 LTC-5723HR, U12 LTC-5723HR, U7 AS1115-BSST, U8 AS1115-BSST, U9 LTC-5723HR

Commit message: updated hardware schimatics for better readability
Other:
- note added: "DISPLAY DRIVER 1"
- note added: "DISPLAY DRIVER 2"
- note added: "DISPLAYS"
- moved on the sheet: C17, C19, R21, R23, TP13, TP14, U8
