File: hardware/reflow.kicad_pcb (KiCad board)
At the start: 2 copper layers, 209 x 130 mm, 119 parts, among them J1 Conn_01x04, J2 Screw_Terminal_01x07, J3 Screw_Terminal_01x02, J4 Screw_Terminal_01x04, J5 Conn_02x03_Odd_Even, J6 Conn_01x07, K1 OZ-SS-112L1, K2 OZ-SS-112L1, K3 SDT-SS-112DM, K4 0J-SS-112LWHF, Q1 RE1C002UNTCL, Q2 RE1C002UNTCL, Q3 RE1C002UNTCL, Q4 RE1C002UNTCL, Q5 RE1C002UNTCL, Q6 RE1C002UNTCL, Q7 RE1C002UNTCL, Q8 RE1C002UNTCL, Q9 RE1C002UNTCL, SW1 UP, SW2 DWN, SW3 ENT, SW4 SW_Push, U1 ESP-12E, U10 LTC-5723HR, U11 LTC-5723HR, U12 LTC-5723HR, U2 AD8495, U3 MC7812BDTRKG, U4 AZ1117CD-3.3TRG1, U5 AZ1117CD-3.3TRG1, U6 PI4IOE5V6416LEX, U7 AS1115-BSST, U8 AS1115-BSST, U9 LTC-5723HR

Commit message: updated kicad files
Routing:
- net +3V3: track 323.5 -> 321.9 mm
Changed lines of the file:
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@@
   (segment (start 90.8 49.8) (end 90.8 45.8) (width 0.5) (layer "B.Cu") (net 2))
   (segment (start 124.2 49) (end 124.2 43.6) (width 0.5) (layer "B.Cu") (net 2))
-  (segment (start 155 91) (end 155 88.4) (width 1) (layer "B.Cu") (net 2))
+  (segment (start 206.8 129) (end 195.6 129) (width 1) (layer "B.Cu") (net 2))
+  (segment (start 195.6 129) (end 155 88.4) (width 1) (layer "B.Cu") (net 2))
   (segment (start 90.8 49.8) (end 90.8 52.8) (width 0.5) (layer "B.Cu") (net 2))
   (segment (start 120.4 87.6) (end 120.4 84.8) (width 0.25) (layer "B.Cu") (net 2))
-  (segment (start 193 129) (end 155 91) (width 1) (layer "B.Cu") (net 2))
-  (segment (start 206.8 129) (end 193 129) (width 1) (layer "B.Cu") (net 2))
   (segment (start 95.6 85.8) (end 95.6 87) (width 0.25) (layer "B.Cu") (net 2))
   (segment (start 123.475 42.875) (end 122.065 42.875) (width 0.5) (layer "B.Cu") (net 2))

Commit message: more hardware revisions
Parts:
- added R24: 660R, Resistor_SMD:R_0603_1608Metric, F.Cu at (69.8, 44.4)
- added R25: 330R, Resistor_SMD:R_0603_1608Metric, F.Cu at (73.2, 44.4)
- added TP16: TestPoint, TestPoint:TestPoint_Pad_D2.0mm, F.Cu at (189.4, 83.2)
- added TP17: TestPoint, TestPoint:TestPoint_Pad_D2.0mm, F.Cu at (160.8, 78.2)
- added TP18: TestPoint, TestPoint:TestPoint_Pad_D2.0mm, F.Cu at (141.8, 77.8)
- added TP19: TestPoint, TestPoint:TestPoint_Pad_D2.0mm, F.Cu at (128.8, 67.8)
- added TP20: TestPoint, TestPoint:TestPoint_Pad_D2.0mm, F.Cu at (76.0, 47.6)
- U1: value ESP-12E -> ESP-12F
- moved TP1 5.37 mm to (68.8, 40.6)
Connections:
- D6 pad 2: /HTR3_C -> /FAN_C
- D8 pad 2: /FAN_C -> /LIGHT_C
- J4 pad 1: FAN_H -> LIGHT_H
- J4 pad 2: HTR3_H -> FAN_H
- K3 pad 6: /HTR3_C -> /FAN_C
- K3 pad 7: HTR3_H -> FAN_H
- K4 pad 6: /FAN_C -> /LIGHT_C
- K4 pad 7: FAN_H -> LIGHT_H
- Q3 pad 1: HTR3_G -> FAN_G
- Q3 pad 3: /HTR3_C -> /FAN_C
- Q4 pad 1: FAN_G -> LIGHT_G
- Q4 pad 3: /FAN_C -> /LIGHT_C
- R3 pad 2: /HTR3_C -> /FAN_C
- R4 pad 2: /FAN_C -> /LIGHT_C
- TP1 pad 1: ESP_ADC -> THERMO_AMP
- U1 pad 20: HTR3_G -> FAN_G
- U2 pad 5: ESP_ADC -> THERMO_AMP
- U2 pad 6: ESP_ADC -> THERMO_AMP
- U6 pad 20: FAN_G -> LIGHT_G
Routing:
- net HTR3_G: track 52.3 -> 0.00 mm
- net FAN_G: track 25.7 -> 52.3 mm, vias 2 -> 0
- net LIGHT_G: track 0.00 -> 25.7 mm, vias 0 -> 2
- net /LIGHT_C: track 0.00 -> 15.2 mm
- net /HTR3_C: track 9.30 -> 0.00 mm
- net /HTR2_C: track 11.0 -> 19.9 mm
- net THERMO_AMP: track 0.00 -> 8.71 mm
- net ESP_ADC: track 37.6 -> 29.4 mm
- net /HTR1_C: track 8.34 -> 16.0 mm
- net /FAN_C: track 10.4 -> 17.9 mm
- net GND: track 626.7 -> 631.0 mm, vias 141 -> 272
- added copper zone on B.Cu, net LIGHT_H
- removed copper zone on B.Cu, net HTR3_H

Commit message: trubbelshooting
Parts:
- TP11, TP14, TP15: moved to F.Cu
- moved TP11 8.05 mm to (94.8, 54.8), turned to 0 degrees
- moved TP15 1.84 mm to (98.4, 101.6), turned to 0 degrees
- moved TP14 1.17 mm to (148.8, 101.6), turned to 0 degrees
Routing:
- net PI4_INT: track 23.8 -> 21.5 mm, vias 1 -> 0
- net +3V3: track 321.9 -> 323.6 mm
- net GND: track 631.0 -> 630.3 mm
- net /DISPLAY/DISP_DVR1_BR: track 16.1 -> 15.5 mm

Commit message: minor hardware refactroing
Parts:
- added R26: 2K2, Resistor_SMD:R_0603_1608Metric, F.Cu at (204.6, 125.8)
- added R27: 660R, Resistor_SMD:R_0603_1608Metric, F.Cu at (208.0, 125.8)
- added R28: 2K2, Resistor_SMD:R_0603_1608Metric, F.Cu at (214.8, 125.8)
- added R29: 660R, Resistor_SMD:R_0603_1608Metric, F.Cu at (211.4, 125.8)
Routing:
- net /POWER/16.33VDC: track 62.6 -> 89.3 mm, vias 0 -> 1
- net GND: track 630.3 -> 643.7 mm, vias 272 -> 274
- net /POWER/10.94VDC: track 83.1 -> 90.1 mm
- net Net-(R28-Pad2): track 0.00 -> 1.75 mm
- net Net-(R26-Pad2): track 0.00 -> 1.75 mm

Commit message: minor hardware refactoring & added firmware fuction
Parts:
- added R30: 330R, Resistor_SMD:R_0603_1608Metric, F.Cu at (112.7, 79.3)
- added R31: 330R, Resistor_SMD:R_0603_1608Metric, F.Cu at (116.2, 79.3)
- added R32: 330R, Resistor_SMD:R_0603_1608Metric, F.Cu at (105.7, 79.3)
- added R33: 330R, Resistor_SMD:R_0603_1608Metric, F.Cu at (102.0, 79.3)
- moved R20 10.0 mm to (109.0, 79.3)
- moved D14 1.85 mm to (109.1, 77.6)
- moved D15 1.85 mm to (112.6, 77.6)
- moved D16 1.85 mm to (116.1, 77.6)
- moved D17 1.85 mm to (105.6, 77.6)
- moved D18 1.85 mm to (102.1, 77.6)
- moved Q5 1.48 mm to (112.7, 75.5)
- moved Q6 1.48 mm to (105.7, 75.5)
- moved Q7 1.48 mm to (109.2, 75.5)
- moved Q8 1.48 mm to (116.2, 75.5)
- moved Q9 1.48 mm to (102.2, 75.5)
Connections:
- D15 pad 2: Net-(D14-Pad2) -> Net-(D15-Pad2)
- D16 pad 2: Net-(D14-Pad2) -> Net-(D16-Pad2)
- D17 pad 2: Net-(D14-Pad2) -> Net-(D17-Pad2)
- D18 pad 2: Net-(D14-Pad2) -> Net-(D18-Pad2)
Routing:
- net Net-(D14-Pad2): track 33.7 -> 1.72 mm
- net +3V3: track 323.6 -> 348.5 mm
- net GND: track 643.7 -> 634.4 mm, vias 274 -> 277
- net /IO/WIFI_OR: track 9.29 -> 7.34 mm
- net Net-(D18-Pad2): track 0.00 -> 1.72 mm
- net Net-(D17-Pad2): track 0.00 -> 1.69 mm
- net Net-(D16-Pad2): track 0.00 -> 1.69 mm
- net Net-(D15-Pad2): track 0.00 -> 1.69 mm
- net /IO/WIFI_G: track 11.5 -> 9.88 mm
- net /IO/RUNNING_R: track 10.2 -> 8.98 mm
- net /IO/WIFI_R: track 8.16 -> 7.18 mm
- net /IO/READY_G: track 7.15 -> 6.24 mm

Commit message: major hardware refctoring to use modern parts that are still being made
Parts:
- removed C11, C8: 10UF, Capacitor_SMD:C_0603_1608Metric
- removed C6, C7: 10000UF, Capacitor_THT:CP_Radial_D35.0mm_P10.00mm_SnapIn
- removed D10, D9: D_Bridge_+-AA, EXTRA:DF01S-TDICT-ND
- removed R26, R28: 2K2, Resistor_SMD:R_0603_1608Metric
- removed R27, R29: 660R, Resistor_SMD:R_0603_1608Metric
- removed TP2, TP3, TP4, TP5, TP6, TP8: TestPoint, TestPoint:TestPoint_Pad_D2.0mm
- removed TRE1: WDB41-18, EXTRA:WDB41-18
- removed U3: MC7812BDTRKG, Package_TO_SOT_SMD:TO-252-3_TabPin2
- added PS1: RAC04-12SK/277, EXTRA:CONV_RAC04-12SK_277, F.Cu at (183.2, 44.4)
- K1, K2: value OZ-SS-112L1 -> J114FL1CS1612VDC; footprint EXTRA:0Z-SS-112L1 -> EXTRA:J114FL1CS1612VDC
- K3: value SDT-SS-112DM -> ALQ112; footprint EXTRA:SDT-SS-112DM -> EXTRA:RELAY_ALQ112
- K4: value 0J-SS-112LWHF -> ALQ112; footprint EXTRA:0J-SS-112LWHF -> EXTRA:RELAY_ALQ112
- moved TP10 118.9 mm to (134.2, 45.2)
- moved C10 114.1 mm to (142.9, 54.6)
- moved C12 114.1 mm to (153.4, 59.1)
- moved C13 114.1 mm to (137.9, 59.1)
- moved C9 114.1 mm to (158.4, 54.6)
- moved D12 114.1 mm to (153.4, 61.1)
- moved D13 114.1 mm to (137.9, 61.1)
- moved R14 114.1 mm to (155.9, 60.1)
- moved R15 114.1 mm to (140.4, 60.1)
- moved U4 114.1 mm to (151.9, 54.6)
- moved U5 114.1 mm to (136.4, 54.6)
- moved R13 92.0 mm to (163.6, 53.2), turned to 180 degrees
- moved D11 90.2 mm to (163.6, 55.2)
- moved TP7 87.1 mm to (143.0, 50.0)
- moved TP9 83.9 mm to (152.6, 65.0)
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Connections:
- C10 pad 1: /POWER/10.94VDC -> +12V
- C9 pad 1: /POWER/10.94VDC -> +12V
- J4 pad 1: LIGHT_H -> HTR1_H
- J4 pad 2: FAN_H -> HTR2_H
- J4 pad 3: HTR2_H -> FAN_H
- J4 pad 4: HTR1_H -> LIGHT_H
- K3 pad 1: 120VAC H -> +12V
- K3 pad 2: +12V -> /FAN_C
- K4 pad 1: 120VAC H -> +12V
- K4 pad 2: +12V -> /LIGHT_C
- TP7 pad 1: /POWER/10.94VDC -> +12V
- U4 pad 3: /POWER/10.94VDC -> +12V
- U5 pad 3: /POWER/10.94VDC -> +12V
Routing:
- net GND: track 634.4 -> 101.1 mm, vias 277 -> 283
- net +3.3VA: track 313.0 -> 122.6 mm, vias 2 -> 0
- net /POWER/10.94VDC: track 90.1 -> 0.00 mm
- net /POWER/16.33VDC: track 89.3 -> 0.00 mm, vias 1 -> 0
- net LIGHT_G: track 25.7 -> 88.8 mm
- net +3V3: track 348.5 -> 285.6 mm, vias 11 -> 4
- net FAN_G: track 52.3 -> 93.8 mm, vias 0 -> 2
- net HTR1_G: track 101.8 -> 71.8 mm
- net LIGHT_H: track 0.00 -> 27.9 mm
- net FAN_H: track 0.00 -> 25.8 mm
- net 10.94VAC N: track 19.1 -> 0.00 mm
- net 10.94VAC H: track 18.4 -> 0.00 mm
- net 16.33 N: track 15.0 -> 0.00 mm
- net 16.33VAC H: track 14.8 -> 0.00 mm
- net +12V: track 169.1 -> 180.1 mm
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- removed copper zone on B.Cu, net FAN_H
- removed copper zone on B.Cu, net LIGHT_H
Other:
- board size 209 x 130 mm -> 305.2 x 234.8 mm
- board text added: "+12 V"
- board text removed: "+12V"
